File: usb2spi.sch (KiCad schematic (older format))
At the start: 15 parts, among them J1 Vout 3.3v 50mA, J2 SPI, J3 Additional, J4 GPIO, J5 Suspend

Commit message: Fix PCB
Parts:
- C1, C2, C4: symbol CP -> CP-RESCUE-usb2spi
- C3: symbol C -> C-RESCUE-usb2spi
- D1: symbol LED -> LED-RESCUE-usb2spi
- R1, R2: symbol R -> R-RESCUE-usb2spi
Changed lines of the file:
@@
 EESchema Schematic File Version 2
+LIBS:usb2spi-rescue
 LIBS:power
 LIBS:device
@@
 LIBS:sp0503baht
 LIBS:usb2spi-cache
-EELAYER 26 0
+EELAYER 25 0
 EELAYER END
 $Descr A4 11693 8268
@@
 $EndComp
 $Comp
-L LED D1
+L LED-RESCUE-usb2spi D1
 U 1 1 5AB247FF
 P 5700 2600
@@
 $EndComp
 $Comp
-L R R2
+L R-RESCUE-usb2spi R2
 U 1 1 5AB24D8C
 P 5350 2600
@@
 $EndComp
 $Comp
-L R R1
+L R-RESCUE-usb2spi R1
 U 1 1 5AB257B7
 P 3200 3300
@@
 $EndComp
 $Comp
-L CP C1
+L CP-RESCUE-usb2spi C1
 U 1 1 5AB25DE3
 P 2600 4150
@@
 $EndComp
 $Comp
-L CP C2
+L CP-RESCUE-usb2spi C2
 U 1 1 5AB25E5E
 P 2900 4150
@@
 $EndComp
 $Comp
-L CP C4
+L CP-RESCUE-usb2spi C4
 U 1 1 5AB25EC9
 P 3500 4150
@@
 $EndComp
 $Comp
-L C C3
+L C-RESCUE-usb2spi C3
 U 1 1 5AB25F26
 P 3200 4150
